Commit message: disable and remove robot arm

File: robots/irlab_summit_xls_std.urdf.xacro (robot description, xacro)
@@ -107,17 +107,17 @@
 		</xacro:hokuyo>
 		<!-- UR5 Arm -->
-		<xacro:ur5_robot prefix="arm_" joint_limits_parameters_file="$(find icclab_summit_xl)/config/joint_limits.yaml"/>
+		<!-- <xacro:ur5_robot prefix="arm_" joint_limits_parameters_file="$(find icclab_summit_xl)/config/joint_limits.yaml"/>
 		<joint name="$(arg prefix)arm_base_joint" type="fixed">
 			<origin xyz="0.255 0 0.275" rpy="0 0 ${PI}" />
 			<parent link="$(arg prefix)base_link" />
 			<child link="arm_base_link" />
-		</joint>
+		</joint> -->
 		<!-- GRIPPER -->
-		<xacro:unless value="$(arg robotiq_gripper)">
+		<!-- <xacro:unless value="$(arg robotiq_gripper)">
 			<xacro:schunk_egp_40 prefix="gripper_" parent="arm_tool0" >
 				 <origin xyz="0.0 0 0.0" rpy="0 0 0" />
 			</xacro:schunk_egp_40>
-  		</xacro:unless>
-		<xacro:if value="$(arg robotiq_gripper)">
+  		</xacro:unless> -->
+		<!-- <xacro:if value="$(arg robotiq_gripper)">
 			<xacro:robotiq_arg2f_140 prefix="gripper_"/>
      				<joint name="gripper_base_joint" type="fixed">
@@ -126,28 +126,28 @@
 					<child link="gripper_robotiq_arg2f_base_link" />
 				</joint>
-		</xacro:if>
+		</xacro:if> -->
 		<!-- Camera on gripper  -->
 		<!-- had to copy and modidy camera to avoid name clash with robotnik defined sensors -->
-		<xacro:sensor_d435_icclab prefix="arm" prefix_topic="summit_xl/arm_camera" parent="gripper_robotiq_arg2f_base_link">
-     		  <origin xyz="0.06 0.0 0.01" rpy="${PI} ${-PI/2} 0"/> <!-- camera on gripper -->
-   		</xacro:sensor_d435_icclab>
+		<!-- <xacro:sensor_d435_icclab prefix="arm" prefix_topic="summit_xl/arm_camera" parent="gripper_robotiq_arg2f_base_link"> -->
+     		  <!-- <origin xyz="0.06 0.0 0.01" rpy="${PI} ${-PI/2} 0"/> camera on gripper -->
+   		<!-- </xacro:sensor_d435_icclab>  -->
 <!--		<sensor_d415_icclab prefix="arm" prefix_topic="arm_camera" parent="arm_wrist_2_link">
      		<origin xyz="0 0.05 0.155" rpy="0 0 ${PI/2}"/>--> <!-- Note the position seems to be wrong in gazebo beacuase we use the d435 mesh file, but it is correct considering the realsize of the camera-->
    		<!--</sensor_d415_icclab>-->
 		<!-- Camera mount -->
-		<xacro:camera_mount prefix="arm" parent="gripper_robotiq_arg2f_base_link">
+		<!-- <xacro:camera_mount prefix="arm" parent="gripper_robotiq_arg2f_base_link"> -->
 			<!-- <origin xyz="-0.005 0.04 0.095" rpy="${PI/2} 0 ${PI}" /> -->
 			 <!--origin xyz="0 0.041 0.09" rpy=" ${PI/2} ${PI/2} ${PI}" /-->  <!-- camera on the one side -->
 			<!--origin xyz="0.005 0.045 0.09" rpy="${PI/2} ${PI} ${PI}" /--><!-- camera on top  -->
-			<origin xyz="0 0 0" rpy="0 0 ${-PI/2}" /><!-- camera on bot  -->
-		</xacro:camera_mount>
+			<!-- <origin xyz="0 0 0" rpy="0 0 ${-PI/2}" />camera on bot  -->
+		<!-- </xacro:camera_mount> -->
 		<!-- Collision box camera cable -->
-		<xacro:collision_box_camera_cable prefix="arm" parent="arm_camera_link">
+		<!-- <xacro:collision_box_camera_cable prefix="arm" parent="arm_camera_link">
 			 <origin xyz="-0.02 -0.08 0" rpy="0 0 0" />
-		</xacro:collision_box_camera_cable>
+		</xacro:collision_box_camera_cable> -->
 		<!-- Collision box wrist 3 -->
-		<xacro:collision_box_wrist3 prefix="arm" parent="arm_wrist_3_link">
+		<!-- <xacro:collision_box_wrist3 prefix="arm" parent="arm_wrist_3_link">
 			 <origin xyz="0 -0.06 0" rpy="0 0 0" />
-		</xacro:collision_box_wrist3>
+		</xacro:collision_box_wrist3>  -->
 		<!-- Collision box wrist 2 -->
 		<!-- <xacro:collision_box_wrist2 prefix="arm" parent="arm_wrist_2_link">
@@ -155,5 +155,5 @@
 		</xacro:collision_box_wrist2>  -->
 		<!-- Collision walls right/left-->
-		<xacro:if value="$(arg collision_walls)">
+		<!-- <xacro:if value="$(arg collision_walls)">
 			<xacro:collision_box_wall prefix="right" parent="summit_xl_base_footprint">
 				 <origin xyz="0 0.8 0.5" rpy="0 0 0" />
@@ -162,5 +162,5 @@
 				 <origin xyz="0 -0.8 0.5" rpy="0 0 0" />
 			</xacro:collision_box_wall>
-		</xacro:if>
+		</xacro:if> -->
    </xacro:macro>
    <xacro:ros_control/>
